File: KiCad_GreenTree/Base/Base.sch (KiCad schematic (older format))
At the start: 23 parts, among them Q1 BCX56, Q2 BCX56, Q3 BCX56, Q4 BCX56, SW1 SW_DPDT_x2, U1 NE555D, U2 NE555D, U3 74HC04, U4 74HC04

Commit message: Verbindung zu Baum
Parts:
- removed U4: 74HC04, Package_SO:SOIC-14W_7.5x9mm_P1.27mm, symbol 74xx:74HC04
- added unit 2 of U3
- C1: footprint Capacitor_SMD:C_01005_0402Metric -> Capacitor_SMD:C_1206_3216Metric_Pad1.33x1.80mm_HandSolder
- C2, C3, C4: footprint Capacitor_SMD:C_01005_0402Metric_Pad0.57x0.30mm_HandSolder -> Capacitor_SMD:C_1206_3216Metric_Pad1.33x1.80mm_HandSolder
- R1, R2, R3, R4, R5, R6: footprint Resistor_SMD:R_01005_0402Metric_Pad0.57x0.30mm_HandSolder -> Resistor_SMD:R_1206_3216Metric_Pad1.30x1.75mm_HandSolder
Connections:
- net at Q2.1 (B), R5.1: now also U3.3
- net at Q4.1 (B): now also U3.4
Changed lines of the file:
@@
 F 0 "R1" H 3020 1496 50  0000 L CNN
 F 1 "R" H 3020 1405 50  0000 L CNN
-F 2 "Resistor_SMD:R_01005_0402Metric_Pad0.57x0.30mm_HandSolder" V 2880 1450 50  0001 C CNN
+F 2 "Resistor_SMD:R_1206_3216Metric_Pad1.30x1.75mm_HandSolder" V 2880 1450 50  0001 C CNN
 F 3 "~" H 2950 1450 50  0001 C CNN
 	1    2950 1450
@@
 F 0 "R2" H 3020 2246 50  0000 L CNN
 F 1 "R" H 3020 2155 50  0000 L CNN
-F 2 "Resistor_SMD:R_01005_0402Metric_Pad0.57x0.30mm_HandSolder" V 2880 2200 50  0001 C CNN
+F 2 "Resistor_SMD:R_1206_3216Metric_Pad1.30x1.75mm_HandSolder" V 2880 2200 50  0001 C CNN
 F 3 "~" H 2950 2200 50  0001 C CNN
 	1    2950 2200
@@
 F 0 "C1" H 965 2346 50  0000 L CNN
 F 1 "10n" H 965 2255 50  0000 L CNN
-F 2 "Capacitor_SMD:C_01005_0402Metric" H 888 2150 50  0001 C CNN
+F 2 "Capacitor_SMD:C_1206_3216Metric_Pad1.33x1.80mm_HandSolder" H 888 2150 50  0001 C CNN
 F 3 "~" H 850 2300 50  0001 C CNN
 	1    850  2300
@@
 F 0 "C3" H 3065 2646 50  0000 L CNN
 F 1 "C" H 3065 2555 50  0000 L CNN
-F 2 "Capacitor_SMD:C_01005_0402Metric_Pad0.57x0.30mm_HandSolder" H 2988 2450 50  0001 C CNN
+F 2 "Capacitor_SMD:C_1206_3216Metric_Pad1.33x1.80mm_HandSolder" H 2988 2450 50  0001 C CNN
 F 3 "~" H 2950 2600 50  0001 C CNN
 	1    2950 2600
@@
 F 0 "R3" H 3020 4346 50  0000 L CNN
 F 1 "R" H 3020 4255 50  0000 L CNN
-F 2 "Resistor_SMD:R_01005_0402Metric_Pad0.57x0.30mm_HandSolder" V 2880 4300 50  0001 C CNN
+F 2 "Resistor_SMD:R_1206_3216Metric_Pad1.30x1.75mm_HandSolder" V 2880 4300 50  0001 C CNN
 F 3 "~" H 2950 4300 50  0001 C CNN
 	1    2950 4300
@@
 F 0 "R4" H 3020 5096 50  0000 L CNN
 F 1 "R" H 3020 5005 50  0000 L CNN
-F 2 "Resistor_SMD:R_01005_0402Metric_Pad0.57x0.30mm_HandSolder" V 2880 5050 50  0001 C CNN
+F 2 "Resistor_SMD:R_1206_3216Metric_Pad1.30x1.75mm_HandSolder" V 2880 5050 50  0001 C CNN
 F 3 "~" H 2950 5050 50  0001 C CNN
 	1    2950 5050
@@
 F 0 "C2" H 965 5196 50  0000 L CNN
 F 1 "10n" H 965 5105 50  0000 L CNN
-F 2 "Capacitor_SMD:C_01005_0402Metric_Pad0.57x0.30mm_HandSolder" H 888 5000 50  0001 C CNN
+F 2 "Capacitor_SMD:C_1206_3216Metric_Pad1.33x1.80mm_HandSolder" H 888 5000 50  0001 C CNN
 F 3 "~" H 850 5150 50  0001 C CNN
 	1    850  5150
@@
 F 0 "C4" H 3065 5496 50  0000 L CNN
 F 1 "C" H 3065 5405 50  0000 L CNN
-F 2 "Capacitor_SMD:C_01005_0402Metric_Pad0.57x0.30mm_HandSolder" H 2988 5300 50  0001 C CNN
+F 2 "Capacitor_SMD:C_1206_3216Metric_Pad1.33x1.80mm_HandSolder" H 2988 5300 50  0001 C CNN
 F 3 "~" H 2950 5450 50  0001 C CNN
 	1    2950 5450
@@
 $EndComp
 $Comp
-L 74xx:74HC04 U4
-U 1 1 6171FDC0
-P 4200 5350
-F 0 "U4" H 4200 5667 50  0000 C CNN
-F 1 "74HC04" H 4200 5576 50  0000 C CNN
-F 2 "Package_SO:SOIC-14W_7.5x9mm_P1.27mm" H 4200 5350 50  0001 C CNN
-F 3 "https://assets.nexperia.com/documents/data-sheet/74HC_HCT04.pdf" H 4200 5350 50  0001 C CNN
-	1    4200 5350
-	1    0    0    -1
-$EndComp
-$Comp
 L Transistor_BJT:BCX56 Q4
 U 1 1 6171FDC6
@@
 	2500 4750 3100 4750
 Wire Wire Line
-	3650 5350 3900 5350
-Wire Wire Line
 	3650 5350 3650 4750
 Connection ~ 3650 4750
@@
 F 0 "R6" V 3093 1900 50  0000 C CNN
 F 1 "R" V 3184 1900 50  0000 C CNN
-F 2 "Resistor_SMD:R_01005_0402Metric_Pad0.57x0.30mm_HandSolder" V 3230 1900 50  0001 C CNN
+F 2 "Resistor_SMD:R_1206_3216Metric_Pad1.30x1.75mm_HandSolder" V 3230 1900 50  0001 C CNN
 F 3 "~" H 3300 1900 50  0001 C CNN
 	1    3300 1900
@@
 F 0 "R5" V 3043 4750 50  0000 C CNN
 F 1 "R" V 3134 4750 50  0000 C CNN
-F 2 "Resistor_SMD:R_01005_0402Metric_Pad0.57x0.30mm_HandSolder" V 3180 4750 50  0001 C CNN
+F 2 "Resistor_SMD:R_1206_3216Metric_Pad1.30x1.75mm_HandSolder" V 3180 4750 50  0001 C CNN
 F 3 "~" H 3250 4750 50  0001 C CNN
 	1    3250 4750
@@
 Wire Wire Line
 	8300 1050 8400 1050
+$Comp
+L 74xx:74HC04 U3
+U 2 1 616C7E94
+P 4200 5350
+F 0 "U3" H 4200 5667 50  0000 C CNN
+F 1 "74HC04" H 4200 5576 50  0000 C CNN
+F 2 "Package_SO:SOIC-14W_7.5x9mm_P1.27mm" H 4200 5350 50  0001 C CNN
+F 3 "https://assets.nexperia.com/documents/data-sheet/74HC_HCT04.pdf" H 4200 5350 50  0001 C CNN
+	2    4200 5350
+	1    0    0    -1
+$EndComp
+Wire Wire Line
+	3650 5350 3900 5350
 $EndSCHEMATC

Commit message: NE555 Layout
Parts:
- added C5, C6: 100n, Capacitor_SMD:C_1206_3216Metric_Pad1.33x1.80mm_HandSolder, symbol Device:C
- SW1: footprint Button_Switch_THT:SW_E-Switch_EG2219_DPDT_Angled -> Bib:Schiebeschalter
Connections:
- net GND: now also C5.2, C6.2
- net VCC: now also C5.1, C6.1
Changed lines of the file:
@@
 	2000 1700 2000 1350
 Wire Wire Line
-	2000 1050 2950 1050
+	2000 1050 2350 1050
 Wire Wire Line
 	2950 1050 2950 1300
@@
 Wire Wire Line
 	2000 4550 2000 4200
-Wire Wire Line
-	2000 3900 2950 3900
 Wire Wire Line
 	2950 3900 2950 4150
@@
 Wire Wire Line
 	9100 1050 9200 1050
-Wire Wire Line
-	10450 950  10450 850
-$Comp
-L power:VCC #PWR0109
-U 1 1 61700D94
-P 10450 850
-F 0 "#PWR0109" H 10450 700 50  0001 C CNN
-F 1 "VCC" H 10465 1023 50  0000 C CNN
-F 2 "" H 10450 850 50  0001 C CNN
-F 3 "" H 10450 850 50  0001 C CNN
-	1    10450 850
-	1    0    0    -1
-$EndComp
 $Comp
 L power:GND #PWR0110
@@
 Text Notes 6500 3050 0    50   ~ 0
 Vorwiderstand vor jeder LED? oder hier?
-$Comp
-L Switch:SW_DPDT_x2 SW1
-U 1 1 6176C986
-P 9950 1050
-F 0 "SW1" H 9950 1335 50  0000 C CNN
-F 1 "SW_DPDT_x2" H 9950 1244 50  0000 C CNN
-F 2 "Button_Switch_THT:SW_E-Switch_EG2219_DPDT_Angled" H 9950 1050 50  0001 C CNN
-F 3 "~" H 9950 1050 50  0001 C CNN
-	1    9950 1050
-	1    0    0    -1
-$EndComp
-Wire Wire Line
-	10150 950  10450 950
 Wire Wire Line
 	9650 1050 9750 1050
@@
 	9650 1050 9500 1050
 Connection ~ 9650 1050
-Wire Wire Line
-	10150 1150 10450 1150
-NoConn ~ 10450 1150
 $Comp
 L Device:R R6
@@
 Wire Wire Line
 	3650 5350 3900 5350
+Wire Wire Line
+	10150 950  10450 950
+$Comp
+L power:VCC #PWR0109
+U 1 1 61700D94
+P 10450 850
+F 0 "#PWR0109" H 10450 700 50  0001 C CNN
+F 1 "VCC" H 10465 1023 50  0000 C CNN
+F 2 "" H 10450 850 50  0001 C CNN
+F 3 "" H 10450 850 50  0001 C CNN
+	1    10450 850
+	1    0    0    -1
+$EndComp
+Wire Wire Line
+	10450 950  10450 850
+NoConn ~ 10450 1150
+Wire Wire Line
+	10150 1150 10450 1150
+$Comp
+L Switch:SW_DPDT_x2 SW1
+U 1 1 6176C986
+P 9950 1050
+F 0 "SW1" H 9950 1335 50  0000 C CNN
+F 1 "SW_DPDT_x2" H 9950 1244 50  0000 C CNN
+F 2 "Bib:Schiebeschalter" H 9950 1050 50  0001 C CNN
+F 3 "~" H 9950 1050 50  0001 C CNN
+	1    9950 1050
+	1    0    0    -1
+$EndComp
+$Comp
+L power:GND #PWR02
+U 1 1 61740863
+P 2350 1550
+F 0 "#PWR02" H 2350 1300 50  0001 C CNN
+F 1 "GND" H 2355 1377 50  0000 C CNN
+F 2 "" H 2350 1550 50  0001 C CNN
+F 3 "" H 2350 1550 50  0001 C CNN
+	1    2350 1550
+	1    0    0    -1
+$EndComp
+$Comp
+L Device:C C6
+U 1 1 6174346D
+P 2350 1300
+F 0 "C6" H 2465 1346 50  0000 L CNN
+F 1 "100n" H 2465 1255 50  0000 L CNN
+F 2 "Capacitor_SMD:C_1206_3216Metric_Pad1.33x1.80mm_HandSolder" H 2388 1150 50  0001 C CNN
+F 3 "~" H 2350 1300 50  0001 C CNN
+	1    2350 1300
+	1    0    0    -1
+$EndComp
+Wire Wire Line
+	2350 1150 2350 1050
+Connection ~ 2350 1050
+Wire Wire Line
+	2350 1050 2950 1050
+Wire Wire Line
+	2350 1450 2350 1550
+$Comp
+L power:GND #PWR01
+U 1 1 6174C201
+P 2300 4400
+F 0 "#PWR01" H 2300 4150 50  0001 C CNN
+F 1 "GND" H 2305 4227 50  0000 C CNN
+F 2 "" H 2300 4400 50  0001 C CNN
+F 3 "" H 2300 4400 50  0001 C CNN
+	1    2300 4400
+	1    0    0    -1
+$EndComp
+$Comp
+L Device:C C5
+U 1 1 6174C207
+P 2300 4150
+F 0 "C5" H 2415 4196 50  0000 L CNN
+F 1 "100n" H 2415 4105 50  0000 L CNN
+F 2 "Capacitor_SMD:C_1206_3216Metric_Pad1.33x1.80mm_HandSolder" H 2338 4000 50  0001 C CNN
+F 3 "~" H 2300 4150 50  0001 C CNN
+	1    2300 4150
+	1    0    0    -1
+$EndComp
+Wire Wire Line
+	2300 4300 2300 4400
+Wire Wire Line
+	2000 3900 2300 3900
+Wire Wire Line
+	2300 4000 2300 3900
+Connection ~ 2300 3900
+Wire Wire Line
+	2300 3900 2950 3900
 $EndSCHEMATC
