File: KiCad_GreenTree/Base/design_versuch_base.kicad_pcb (KiCad board)
At the start: 2 copper layers, 65 x 62.2 mm, 46 parts, among them Q1 BCX56, Q2 BCX56, Q3 BCX56, Q4 BCX56, SW1 SW_DPDT_x2, U1 NE555D, U2 NE555D, U3 74HC04, U4 L78L05_TO92

Commit message: optimierung der Leitungen
Routing:
- net +9V: track 80.2 -> 85.1 mm
- net GND: track 252.7 -> 253.3 mm
