File: KiCad_GreenTree/BaumOben/_autosave-BaumOben.kicad_pcb (KiCad board)
At the start: 2 copper layers, 73.4 x 99.4 mm, 1 part

Commit message: Schaltplan oben
Schaltplan oben fertig und Layout angefangen
Parts:
- removed G***: LOGO, grafics:Baum2.0
- added DB1: LED, Diode_SMD:D_0603_1608Metric_Pad1.05x0.95mm_HandSolder, F.Cu at (191.0, 95.9)
- added DB2: LED, Diode_SMD:D_0603_1608Metric_Pad1.05x0.95mm_HandSolder, F.Cu at (184.0, 95.9)
- added DB3: LED, Diode_SMD:D_0603_1608Metric_Pad1.05x0.95mm_HandSolder, F.Cu at (191.5, 101.0)
- added DB4: LED, Diode_SMD:D_0603_1608Metric_Pad1.05x0.95mm_HandSolder, F.Cu at (184.8, 101.2)
- added DB5: LED, Diode_SMD:D_0603_1608Metric_Pad1.05x0.95mm_HandSolder, F.Cu at (191.4, 106.2)
- added DB6: LED, Diode_SMD:D_0603_1608Metric_Pad1.05x0.95mm_HandSolder, F.Cu at (185.1, 106.1)
- added DB7: LED, Diode_SMD:D_0603_1608Metric_Pad1.05x0.95mm_HandSolder, F.Cu at (191.8, 112.9)
- added DB8: LED, Diode_SMD:D_0603_1608Metric_Pad1.05x0.95mm_HandSolder, F.Cu at (185.9, 112.7)
- added DG1: LED, Diode_SMD:D_0805_2012Metric_Pad1.15x1.40mm_HandSolder, F.Cu at (186.9, 61.7)
- added DG2: LED, Diode_SMD:D_0805_2012Metric_Pad1.15x1.40mm_HandSolder, F.Cu at (178.0, 62.7)
- added DG3: LED, Diode_SMD:D_0805_2012Metric_Pad1.15x1.40mm_HandSolder, F.Cu at (169.3, 62.3)
- added DG4: LED, Diode_SMD:D_0805_2012Metric_Pad1.15x1.40mm_HandSolder, F.Cu at (161.4, 62.4)
- added DG5: LED, Diode_SMD:D_0805_2012Metric_Pad1.15x1.40mm_HandSolder, F.Cu at (193.5, 67.2)
- added DG6: LED, Diode_SMD:D_0805_2012Metric_Pad1.15x1.40mm_HandSolder, F.Cu at (187.9, 67.3)
- added DG7: LED, Diode_SMD:D_0805_2012Metric_Pad1.15x1.40mm_HandSolder, F.Cu at (178.9, 68.6)
- added DG8: LED, Diode_SMD:D_0805_2012Metric_Pad1.15x1.40mm_HandSolder, F.Cu at (169.4, 69.0)
- added DR1: LED, Diode_SMD:D_0805_2012Metric_Pad1.15x1.40mm_HandSolder, F.Cu at (76.8, 125.3)
- added DR2: LED, Diode_SMD:D_0805_2012Metric_Pad1.15x1.40mm_HandSolder, B.Cu at (81.8, 116.3)
- added DR3: LED, Diode_SMD:D_0805_2012Metric_Pad1.15x1.40mm_HandSolder, F.Cu at (104.6, 64.7)
- added DR4: LED, Diode_SMD:D_0805_2012Metric_Pad1.15x1.40mm_HandSolder, B.Cu at (107.6, 67.4)
- added DR5: LED, Diode_SMD:D_0805_2012Metric_Pad1.15x1.40mm_HandSolder, F.Cu at (117.0, 115.1)
- added DR6: LED, Diode_SMD:D_0805_2012Metric_Pad1.15x1.40mm_HandSolder, B.Cu at (111.3, 107.2)
- added DR7: LED, Diode_SMD:D_0805_2012Metric_Pad1.15x1.40mm_HandSolder, F.Cu at (86.7, 90.4)
- added DR8: LED, Diode_SMD:D_0805_2012Metric_Pad1.15x1.40mm_HandSolder, B.Cu at (92.5, 113.1)
- added DY1: LED, Diode_SMD:D_0805_2012Metric_Pad1.15x1.40mm_HandSolder, F.Cu at (87.6, 120.5)
- added DY2: LED, Diode_SMD:D_0805_2012Metric_Pad1.15x1.40mm_HandSolder, B.Cu at (83.4, 96.3)
- added DY3: LED, Diode_SMD:D_0805_2012Metric_Pad1.15x1.40mm_HandSolder, B.Cu at (92.6, 84.8)
- added DY4: LED, Diode_SMD:D_0805_2012Metric_Pad1.15x1.40mm_HandSolder, F.Cu at (111.6, 89.8)
- added DY5: LED, Diode_SMD:D_0805_2012Metric_Pad1.15x1.40mm_HandSolder, B.Cu at (117.7, 124.6)
- added DY6: LED, Diode_SMD:D_0805_2012Metric_Pad1.15x1.40mm_HandSolder, F.Cu at (109.3, 71.1)
- added DY7: LED, Diode_SMD:D_0805_2012Metric_Pad1.15x1.40mm_HandSolder, B.Cu at (95.3, 69.4)
- added DY8: LED, Diode_SMD:D_0805_2012Metric_Pad1.15x1.40mm_HandSolder, F.Cu at (93.3, 98.9)
- added R1: 50, Resistor_SMD:R_0805_2012Metric_Pad1.15x1.40mm_HandSolder, F.Cu at (111.3, 95.3)
- added R10: 88, Resistor_SMD:R_0805_2012Metric_Pad1.15x1.40mm_HandSolder, F.Cu at (180.0, 112.8)
- added R2: 50, Resistor_SMD:R_0805_2012Metric_Pad1.15x1.40mm_HandSolder, B.Cu at (96.6, 103.0)
- added R3: 50, Resistor_SMD:R_0805_2012Metric_Pad1.15x1.40mm_HandSolder, F.Cu at (105.8, 74.3)
- added R4: 50, Resistor_SMD:R_0805_2012Metric_Pad1.15x1.40mm_HandSolder, B.Cu at (93.5, 117.3)
- added R5: 10, Resistor_SMD:R_0805_2012Metric_Pad1.15x1.40mm_HandSolder, F.Cu at (156.2, 62.9)
- added R6: 10, Resistor_SMD:R_0805_2012Metric_Pad1.15x1.40mm_HandSolder, F.Cu at (163.1, 68.9)
- added R7: 88, Resistor_SMD:R_0805_2012Metric_Pad1.15x1.40mm_HandSolder, F.Cu at (178.7, 95.9)
- added R8: 88, Resistor_SMD:R_0805_2012Metric_Pad1.15x1.40mm_HandSolder, F.Cu at (179.6, 101.2)
- added R9: 88, Resistor_SMD:R_0805_2012Metric_Pad1.15x1.40mm_HandSolder, F.Cu at (179.6, 106.2)
Routing:
- net Net-(DR2-Pad1): track 0.00 -> 68.9 mm, vias 0 -> 1
- net Net-(DY5-Pad1): track 0.00 -> 59.7 mm, vias 0 -> 1
- net Takt_9V: track 0.00 -> 44.6 mm
- net Net-(DY7-Pad1): track 0.00 -> 29.5 mm, vias 0 -> 1
- net Takt_invertiert_9V: track 0.00 -> 29.2 mm
- net Net-(DY1-Pad1): track 0.00 -> 26.1 mm, vias 0 -> 1
- net Net-(DY3-Pad1): track 0.00 -> 19.0 mm, vias 0 -> 1
- net Net-(DY2-Pad1): track 0.00 -> 15.4 mm
- net Net-(DR4-Pad1): track 0.00 -> 12.8 mm, vias 0 -> 1
- net Net-(DY6-Pad1): track 0.00 -> 12.7 mm, vias 0 -> 1
- net Net-(DR1-Pad1): track 0.00 -> 11.1 mm, vias 0 -> 1
- net Net-(DY8-Pad1): track 0.00 -> 6.96 mm, vias 0 -> 1
- net Net-(DY4-Pad1): track 0.00 -> 5.06 mm
- net Net-(DR3-Pad1): track 0.00 -> 4.59 mm, vias 0 -> 1
- added copper zone on B.Cu, net GND
- added copper zone on F.Cu, net GND
- added copper zone on B.Cu, net Takt_9V
- added copper zone on F.Cu, net Takt_9V
- added copper zone on B.Cu, net Takt_invertiert_9V
- added copper zone on F.Cu, net Takt_invertiert_9V
Other:
- outline, holes or cut-outs redrawn

Commit message: layout weiter gemacht
Parts:
- DB1, DB3, DG2, DG4, DG6, DG8, R5, R6: moved to B.Cu
- moved DB1 106.4 mm to (89.7, 128.5)
- moved DG1 94.1 mm to (94.6, 80.1)
- moved DB2 89.6 mm to (95.4, 109.5)
- moved DG5 89.4 mm to (125.0, 124.5)
- moved DB3 89.1 mm to (104.8, 80.1), turned to 90 degrees
- moved DG7 88.7 mm to (90.3, 73.0), turned to 180 degrees
- moved R5 87.5 mm to (105.0, 133.9), turned to 180 degrees
- moved DG4 87.3 mm to (106.2, 130.1), turned to 180 degrees
- moved R7 84.7 mm to (95.6, 112.1)
- moved DB4 83.7 mm to (104.8, 125.9), turned to 90 degrees
- moved DG3 83.3 mm to (107.1, 117.8)
- moved DG6 79.3 mm to (110.7, 85.8)
- moved R8 74.3 mm to (109.5, 125.9), turned to 90 degrees
- moved DG8 73.1 mm to (96.6, 75.1), turned to 90 degrees
- moved DG2 67.1 mm to (118.5, 93.7), turned to 180 degrees
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Routing:
- net Net-(DG5-Pad1): track 0.00 -> 49.5 mm, vias 0 -> 1
- net Takt_9V: track 44.6 -> 90.3 mm, vias 0 -> 2
- net Net-(DG6-Pad1): track 0.00 -> 40.1 mm, vias 0 -> 1
- net Net-(DR6-Pad1): track 0.00 -> 39.9 mm, vias 0 -> 1
- net Net-(DG1-Pad1): track 0.00 -> 37.2 mm, vias 0 -> 1
- net Net-(DG2-Pad1): track 0.00 -> 28.8 mm, vias 0 -> 1
- net Takt_invertiert_9V: track 29.2 -> 54.8 mm, vias 0 -> 2
- net Net-(DR7-Pad1): track 0.00 -> 25.1 mm, vias 0 -> 1
- net Net-(DG3-Pad1): track 0.00 -> 12.7 mm, vias 0 -> 1
- net Net-(DR5-Pad1): track 0.00 -> 10.2 mm, vias 0 -> 1
- net Net-(DG7-Pad1): track 0.00 -> 5.73 mm, vias 0 -> 1
- net Net-(DB4-Pad1): track 0.00 -> 4.70 mm
- net Net-(DR8-Pad1): track 0.00 -> 4.65 mm
- net Net-(DG4-Pad1): track 0.00 -> 4.31 mm
- net Net-(DG8-Pad1): track 0.00 -> 3.37 mm
