File: KiCad_GreenTree/BaumOben/_autosave-BaumOben.sch (KiCad schematic (older format))
At the start: 42 parts

Commit message: bis auf silk fertig
baum unten fertig gemacht und Beinchen gekürzt
Parts:
- added C1, C2: 100n, Capacitor_SMD:C_1206_3216Metric_Pad1.42x1.75mm_HandSolder, symbol Device:C
Connections:
- wire segments 56 -> 72
Changed lines of the file:
@@
 $EndDescr
 Wire Wire Line
-	2000 1500 3500 1500
-Wire Wire Line
-	2000 2000 3500 2000
-Wire Wire Line
-	2000 2500 3500 2500
-Wire Wire Line
-	2000 3000 3500 3000
+	2000 1500 2150 1500
+Wire Wire Line
+	2000 2000 2150 2000
+Wire Wire Line
+	2000 2500 2150 2500
+Wire Wire Line
+	2000 3000 2150 3000
 Text GLabel 2000 1500 0    50   Input ~ 0
 Takt_9V
@@
 	1    0    0    -1
 $EndComp
+$Comp
+L power:PWR_FLAG #FLG0101
+U 1 1 617037BB
+P 2150 1450
+F 0 "#FLG0101" H 2150 1525 50  0001 C CNN
+F 1 "PWR_FLAG" H 2150 1623 50  0000 C CNN
+F 2 "" H 2150 1450 50  0001 C CNN
+F 3 "~" H 2150 1450 50  0001 C CNN
+	1    2150 1450
+	1    0    0    -1
+$EndComp
+$Comp
+L power:PWR_FLAG #FLG0102
+U 1 1 6170533C
+P 2150 1950
+F 0 "#FLG0102" H 2150 2025 50  0001 C CNN
+F 1 "PWR_FLAG" H 2150 2123 50  0000 C CNN
+F 2 "" H 2150 1950 50  0001 C CNN
+F 3 "~" H 2150 1950 50  0001 C CNN
+	1    2150 1950
+	1    0    0    -1
+$EndComp
+$Comp
+L power:PWR_FLAG #FLG0103
+U 1 1 617063A7
+P 2150 2450
+F 0 "#FLG0103" H 2150 2525 50  0001 C CNN
+F 1 "PWR_FLAG" H 2150 2623 50  0000 C CNN
+F 2 "" H 2150 2450 50  0001 C CNN
+F 3 "~" H 2150 2450 50  0001 C CNN
+	1    2150 2450
+	1    0    0    -1
+$EndComp
+$Comp
+L power:PWR_FLAG #FLG0104
+U 1 1 6170749A
+P 2150 2950
+F 0 "#FLG0104" H 2150 3025 50  0001 C CNN
+F 1 "PWR_FLAG" H 2150 3123 50  0000 C CNN
+F 2 "" H 2150 2950 50  0001 C CNN
+F 3 "~" H 2150 2950 50  0001 C CNN
+	1    2150 2950
+	1    0    0    -1
+$EndComp
+Wire Wire Line
+	2150 2950 2150 3000
+Connection ~ 2150 3000
+Wire Wire Line
+	2150 3000 2750 3000
+Wire Wire Line
+	2150 2450 2150 2500
+Connection ~ 2150 2500
+Wire Wire Line
+	2150 2500 2750 2500
+Wire Wire Line
+	2150 1950 2150 2000
+Connection ~ 2150 2000
+Wire Wire Line
+	2150 2000 2750 2000
+Wire Wire Line
+	2150 1450 2150 1500
+Connection ~ 2150 1500
+Wire Wire Line
+	2150 1500 2750 1500
+$Comp
+L Device:C C1
+U 1 1 6171479C
+P 2750 1750
+F 0 "C1" H 2865 1796 50  0000 L CNN
+F 1 "100n" H 2865 1705 50  0000 L CNN
+F 2 "Capacitor_SMD:C_1206_3216Metric_Pad1.42x1.75mm_HandSolder" H 2788 1600 50  0001 C CNN
+F 3 "~" H 2750 1750 50  0001 C CNN
+	1    2750 1750
+	1    0    0    -1
+$EndComp
+$Comp
+L Device:C C2
+U 1 1 6171504D
+P 2750 2750
+F 0 "C2" H 2865 2796 50  0000 L CNN
+F 1 "100n" H 2865 2705 50  0000 L CNN
+F 2 "Capacitor_SMD:C_1206_3216Metric_Pad1.42x1.75mm_HandSolder" H 2788 2600 50  0001 C CNN
+F 3 "~" H 2750 2750 50  0001 C CNN
+	1    2750 2750
+	1    0    0    -1
+$EndComp
+Wire Wire Line
+	2750 1600 2750 1500
+Connection ~ 2750 1500
+Wire Wire Line
+	2750 1500 3500 1500
+Wire Wire Line
+	2750 1900 2750 2000
+Connection ~ 2750 2000
+Wire Wire Line
+	2750 2000 3500 2000
+Wire Wire Line
+	2750 2600 2750 2500
+Connection ~ 2750 2500
+Wire Wire Line
+	2750 2500 3500 2500
+Wire Wire Line
+	2750 2900 2750 3000
+Connection ~ 2750 3000
+Wire Wire Line
+	2750 3000 3500 3000
 $EndSCHEMATC

Commit message: footprint auf 0805
Parts:
- C1, C2: footprint Capacitor_SMD:C_1206_3216Metric_Pad1.42x1.75mm_HandSolder -> Capacitor_SMD:C_0805_2012Metric_Pad1.15x1.40mm_HandSolder
Changed lines of the file:
@@
 F 0 "C1" H 2865 1796 50  0000 L CNN
 F 1 "100n" H 2865 1705 50  0000 L CNN
-F 2 "Capacitor_SMD:C_1206_3216Metric_Pad1.42x1.75mm_HandSolder" H 2788 1600 50  0001 C CNN
+F 2 "Capacitor_SMD:C_0805_2012Metric_Pad1.15x1.40mm_HandSolder" H 2788 1600 50  0001 C CNN
 F 3 "~" H 2750 1750 50  0001 C CNN
 	1    2750 1750
@@
 F 0 "C2" H 2865 2796 50  0000 L CNN
 F 1 "100n" H 2865 2705 50  0000 L CNN
-F 2 "Capacitor_SMD:C_1206_3216Metric_Pad1.42x1.75mm_HandSolder" H 2788 2600 50  0001 C CNN
+F 2 "Capacitor_SMD:C_0805_2012Metric_Pad1.15x1.40mm_HandSolder" H 2788 2600 50  0001 C CNN
 F 3 "~" H 2750 2750 50  0001 C CNN
 	1    2750 2750
