File: KiCad_GreenTree/BaumUnten/BaumUnten.sch (KiCad schematic (older format))
At the start: 44 parts

Commit message: footprint auf 0805
Parts:
- C1, C2: footprint Capacitor_SMD:C_1206_3216Metric_Pad1.42x1.75mm_HandSolder -> Capacitor_SMD:C_0805_2012Metric_Pad1.15x1.40mm_HandSolder
Changed lines of the file:
@@
 F 0 "C1" H 2815 1796 50  0000 L CNN
 F 1 "100n" H 2815 1705 50  0000 L CNN
-F 2 "Capacitor_SMD:C_1206_3216Metric_Pad1.42x1.75mm_HandSolder" H 2738 1600 50  0001 C CNN
+F 2 "Capacitor_SMD:C_0805_2012Metric_Pad1.15x1.40mm_HandSolder" H 2738 1600 50  0001 C CNN
 F 3 "~" H 2700 1750 50  0001 C CNN
 	1    2700 1750
@@
 F 0 "C2" H 2815 2796 50  0000 L CNN
 F 1 "100n" H 2815 2705 50  0000 L CNN
-F 2 "Capacitor_SMD:C_1206_3216Metric_Pad1.42x1.75mm_HandSolder" H 2738 2600 50  0001 C CNN
+F 2 "Capacitor_SMD:C_0805_2012Metric_Pad1.15x1.40mm_HandSolder" H 2738 2600 50  0001 C CNN
 F 3 "~" H 2700 2750 50  0001 C CNN
 	1    2700 2750
